File: ulay65.kicad_sch (KiCad schematic)
At the start: 83 parts

Commit message: Finished most of the schematic
This upload is mainly a buffer for myself to be able to revert back.
Parts:
- removed MX? (x76): MX-NoLED, symbol MX_Alps_Hybrid:MX-NoLED
- added '1, ,1, .1, /1, ;1, A1, B1, Bspc1, C1, Cap1, Down1, E1, Enter1, Equal1, Esc40, F1, G1, H1, I1, J1, K1, L1, LSHIFT (x2), L_Brc1, Lalt1, Lalt2, Lctrl1, Lctrl2, Left1, LetterD_1, M1, Macro1, Macro2, Macro3, Menu1, Minus1, N1, Num_1, Num_10, Num_2, Num_3, Num_4, Num_5, Num_6, Num_7, Num_8, Num_9, O1, P1, Q1, R1, R_Brc1, Right1, S1, T1, Tab1, U1, Up1, V1, W1, Win1, X1, Y1, Z1, \1: MX-NoLED, symbol MX_Alps_Hybrid:MX-NoLED
- added D1, D10, D11, D12, D13, D14, D15, D17, D18, D19, D2, D20, D21, D22, D23, D24, D25, D26, D27, D28, D29, D3, D30, D33, D34, D35, D36, D37, D38, D39, D4, D40, D41, D42, D43, D44, D46, D49, D5, D50, D51, D52, D53, D54, D55, D56, D57, D58, D59, D6, D61, D62, D65, D66, D67, D7, D71, D74, D75, D76, D77, D78, D8, D9, D? (x4): D_Small, symbol Device:D_Small
- gave numbers to parts that had none: 7
Connections:
- net COL0: now also Cap1.1 (COL), LSHIFT.1 (COL), Lctrl1.1 (COL), Tab1.1 (COL)
- net COL1: now also A1.1 (COL), Num_1.1 (COL), Q1.1 (COL), Win1.1 (COL), Z1.1 (COL)
- net COL10: now also /1.1 (COL), ;1.1 (COL), Menu1.1 (COL), Num_10.1 (COL), P1.1 (COL)
- net COL11: now also '1.1 (COL), L_Brc1.1 (COL), Lctrl2.1 (COL), Minus1.1 (COL)
- net COL12: now also Equal1.1 (COL), LSHIFT.1 (COL), Left1.1 (COL), R_Brc1.1 (COL)
- net COL13: now also Bspc1.1 (COL), Down1.1 (COL), Enter1.1 (COL), Up1.1 (COL), \1.1 (COL)
- net COL14: now also Macro1.1 (COL), Macro2.1 (COL), Macro3.1 (COL), Right1.1 (COL)
- net COL2: now also Lalt1.1 (COL), Num_2.1 (COL), S1.1 (COL), W1.1 (COL), X1.1 (COL)
- net COL3: now also C1.1 (COL), E1.1 (COL), LetterD_1.1 (COL), Num_3.1 (COL)
- net COL4: now also F1.1 (COL), Num_4.1 (COL), R1.1 (COL), V1.1 (COL)
- net COL5: now also B1.1 (COL), G1.1 (COL), Num_5.1 (COL), T1.1 (COL)
- net COL6: now also Esc40.1 (COL), H1.1 (COL), N1.1 (COL), Num_6.1 (COL), Y1.1 (COL)
- net COL7: now also J1.1 (COL), M1.1 (COL), Num_7.1 (COL), U1.1 (COL)
- net COL8: now also ,1.1 (COL), I1.1 (COL), K1.1 (COL), Num_8.1 (COL)
- net COL9: now also .1.1 (COL), L1.1 (COL), Lalt2.1 (COL), Num_9.1 (COL), O1.1 (COL)
- net GND: now also Enc1.C
- net ROW0: now also D10.1 (K), D11.1 (K), D12.1 (K), D13.1 (K), D14.1 (K), D15.1 (K), D2.1 (K), D3.1 (K), D4.1 (K), D5.1 (K), D6.1 (K), D7.1 (K), D8.1 (K), D9.1 (K); no longer Esc1.2 (ROW)
- net ROW1: now also D17.1 (K), D18.1 (K), D19.1 (K), D20.1 (K), D21.1 (K), D22.1 (K), D23.1 (K), D24.1 (K), D25.1 (K), D26.1 (K), D27.1 (K), D28.1 (K), D29.1 (K), D30.1 (K), D?.1 (K)
- net ROW2: now also D33.1 (K), D34.1 (K), D35.1 (K), D36.1 (K), D37.1 (K), D38.1 (K), D39.1 (K), D40.1 (K), D41.1 (K), D42.1 (K), D43.1 (K), D44.1 (K), D46.1 (K), D?.1 (K)
- net ROW3: now also D49.1 (K), D50.1 (K), D51.1 (K), D52.1 (K), D53.1 (K), D54.1 (K), D55.1 (K), D56.1 (K), D57.1 (K), D58.1 (K), D59.1 (K), D61.1 (K), D62.1 (K), D?.1 (K)
- net ROW4: now also D65.1 (K), D66.1 (K), D67.1 (K), D71.1 (K), D74.1 (K), D75.1 (K), D76.1 (K), D77.1 (K), D78.1 (K), D?.1 (K)
- net EC11-A: now reaches Enc1.A
- net EC11-B: now reaches Enc1.B
- net RS1: now reaches Enc1.S1
- net RS2: now reaches Enc1.S2
- new net: D71.2 (A), Esc40.2 (ROW)
- new net: ,1.2 (ROW), D57.2 (A)
- new net: D3.2 (A), Num_1.2 (ROW)
- new net: D?.2 (A), Macro3.2 (ROW)
- new net: D24.2 (A), U1.2 (ROW)
- new net: D26.2 (A), O1.2 (ROW)
- new net: D38.2 (A), G1.2 (ROW)
- new net: D8.2 (A), Num_6.2 (ROW)
- new net: D76.2 (A), Lctrl2.2 (ROW)
- new net: D39.2 (A), H1.2 (ROW)
- new net: D5.2 (A), Num_3.2 (ROW)
- new net: D77.2 (A), Left1.2 (ROW)
- new net: Bspc1.2 (ROW), D15.2 (A)
- new net: D40.2 (A), J1.2 (ROW)
- new net: D42.2 (A), L1.2 (ROW)
- new net: D4.2 (A), Num_2.2 (ROW)
- new net: D49.2 (A), LSHIFT.2 (ROW)
- new net: D21.2 (A), R1.2 (ROW)
- new net: D37.2 (A), F1.2 (ROW)
- new net: C1.2 (ROW), D52.2 (A)
- new net: D62.2 (A), Up1.2 (ROW)
- new net: D?.2 (A), Macro2.2 (ROW)
- new net: ;1.2 (ROW), D43.2 (A)
- new net: D23.2 (A), Y1.2 (ROW)
- new net: D18.2 (A), Q1.2 (ROW)
- new net: D53.2 (A), V1.2 (ROW)
- new net: D30.2 (A), \1.2 (ROW)
- new net: '1.2 (ROW), D44.2 (A)
- new net: D55.2 (A), N1.2 (ROW)
- new net: D22.2 (A), T1.2 (ROW)
- new net: D46.2 (A), Enter1.2 (ROW)
- new net: D36.2 (A), LetterD_1.2 (ROW)
- new net: /1.2 (ROW), D59.2 (A)
- new net: D19.2 (A), W1.2 (ROW)
- new net: D9.2 (A), Num_7.2 (ROW)
- new net: D14.2 (A), Equal1.2 (ROW)
- new net: D11.2 (A), Num_9.2 (ROW)
- new net: D75.2 (A), Menu1.2 (ROW)
- new net: A1.2 (ROW), D34.2 (A)
- new net: D67.2 (A), Lalt1.2 (ROW)
- new net: .1.2 (ROW), D58.2 (A)
- new net: B1.2 (ROW), D54.2 (A)
- new net: D66.2 (A), Win1.2 (ROW)
- new net: D20.2 (A), E1.2 (ROW)
- new net: D7.2 (A), Num_5.2 (ROW)
- new net: D17.2 (A), Tab1.2 (ROW)
- new net: D29.2 (A), R_Brc1.2 (ROW)
- new net: D35.2 (A), S1.2 (ROW)
- new net: D27.2 (A), P1.2 (ROW)
- new net: D12.2 (A), Num_10.2 (ROW)
- new net: D13.2 (A), Minus1.2 (ROW)
- new net: D61.2 (A), LSHIFT.2 (ROW)
- new net: D65.2 (A), Lctrl1.2 (ROW)
- new net: D?.2 (A), Macro1.2 (ROW)
- new net: D50.2 (A), Z1.2 (ROW)
- new net: D6.2 (A), Num_4.2 (ROW)
- new net: Cap1.2 (ROW), D33.2 (A)
- new net: D25.2 (A), I1.2 (ROW)
- new net: D56.2 (A), M1.2 (ROW)
- new net: D78.2 (A), Down1.2 (ROW)
- new net: D28.2 (A), L_Brc1.2 (ROW)
- new net: D41.2 (A), K1.2 (ROW)
- new net: D10.2 (A), Num_8.2 (ROW)
- new net: D51.2 (A), X1.2 (ROW)
- new net: D2.2 (A), Esc1.2 (ROW)
- new net: D?.2 (A), Right1.2 (ROW)
- new net: D74.2 (A), Lalt2.2 (ROW)
Other:
- moved on the sheet: Enc1, Esc1, F1, U3, USB1
